File: Phone_EE445L/Phone_EE445L.brd (EAGLE design)
At the start: 102 x 70 mm, 58 parts, among them IC1 LM4041CILPRCLP, Q1 NX5032GA, U2 TLV5616, U3 TPA751

Commit message: Added Ground Plane on PCB Artist Version
Parts:
- moved U$3 264.8 mm to (21.4, 57.5), turned to 180 degrees
- moved U$2 222.2 mm to (46.9, 4.25)
- moved JP2 66.4 mm to (-7.27, 37.9), turned to 180 degrees
- moved JP1 58.9 mm to (19.1, 33.4), turned to 90 degrees
- moved U$1 2.24 mm to (91.9, 33.6)
- moved U1 0.89 mm to (47.4, 35.4), turned to 135 degrees
Other:
- board size 102 x 70 mm -> 97.7 x 67.2 mm

Commit message: Continued finishing final board
Parts:
- removed JP1: (no value), EE445L:1X05
- removed JP2, JP3, JP4, JP6, JP7: (no value), EE445L:1X02
- removed JP5: (no value), EE445L:1X03
- removed TP1, TP2, TP3, TP4, TP5: TP_KEYSTONE500X, EE445L:P1.1MM
- added 3.3V, CCS, CS0, CS1, DC0, FSS1, HIB, KEY, MISO0, MOSI0, MOSI1, NS, PS, RI, RST0, RSTG, SCK0, SCL2, SCLK1, SDA2, SDD, U0RX, U0TX, U2RX, U2TX, U6RX, U6TX, VDDC, VREFA, WAKE, X+, X-, Y+, Y-: TP_KEYSTONE500X, EE445L:P1.1MM
- added JTAG: (no value), EE445L:1X05
- added LCD-PWR: (no value), EE445L:1X03
- added LITE, PWR, SPKDAC, SPKR, UART0: (no value), EE445L:1X02
- added SW1: (no value), EE445L:PWRBUTTON
- S1: value (none) -> MOMENTARY-SWITCH-SPST-SMD-6.2MM-TALL; device EE445L:B3F-10XX -> SparkFun-Switches:TACTILE_SWITCH_SMD_6.2MM_TALL
- moved R14 336.4 mm to (47.5, 2.22)
- moved R13 330.0 mm to (29.5, 13.9)
- moved R9 325.8 mm to (7.30, 64.3), turned to 180 degrees
- moved R10 324.7 mm to (45.8, 10.1), turned to 90 degrees
- moved R12 324.1 mm to (30.6, 11.0), turned to 270 degrees
- moved MICRO-USB 321.4 mm to (6.10, 10.7), turned to 270 degrees
- moved C16 320.4 mm to (50.4, 13.0)
- moved D1 319.5 mm to (7.30, 62.1)
- moved C13 319.1 mm to (14.3, 62.0), turned to 180 degrees
- moved R11 316.3 mm to (30.5, 6.37), turned to 270 degrees
- moved C14 304.5 mm to (45.8, 6.33), turned to 270 degrees
- moved IC1 304.4 mm to (26.1, 9.68), turned to 270 degrees
- moved C12 302.3 mm to (14.4, 47.1), turned to 180 degrees
- moved C15 301.8 mm to (40.5, 2.27), turned to 180 degrees
- moved U$4 298.1 mm to (16.2, 54.5), turned to 90 degrees
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Connections:
- net N$14 renamed HPF
- net N$15 renamed AMPIN
- net N$9 renamed DACOUT
- removed net GNDA: C1.2, C2.2, C3.2, C4.2, U1.10, U1.114, U1.17, U1.48, U1.55, U1.58, U1.80
- removed net N$2: C1.1, C2.1, C3.1, C4.1, JP2.1, R2.2, R3.1, U1.101, U1.113, U1.122, U1.16, U1.26, U1.28, U1.39, U1.47, U1.51, U1.52, U1.69, U1.7, U1.79, U1.8, U1.90
- removed net N$3: R3.2, R4.1, R5.1, TP2.TP
- removed net N$6: JP5.2, U$1.2
- new net 5VIN: MICRO-USB.1, PWR.1, SW1.1
- new net LCDPWR: LCD-PWR.2, U$1.2
- new net WAKEVDD: 3.3V.TP, R3.2, R4.1, R5.1
- net +3V3: now also C1.1, C2.1, C3.1, C4.1, LCD-PWR.3, LITE.2, R2.2, R3.1, U1.101, U1.113, U1.122, U1.16, U1.26, U1.28, U1.39, U1.47, U1.51, U1.52, U1.69, U1.7, U1.79, U1.8, U1.90; no longer JP2.2, JP5.3, JP6.2
- net +5V: now also LCD-PWR.1, PWR.2, SW1.6; no longer JP5.1, MICRO-USB.1
- net GND: now also C1.2, C2.2, C3.2, C4.2, JTAG.5, S1.B2, SW1.3, SW1.7, U1.10, U1.114, U1.17, U1.48, U1.55, U1.58, U1.80; no longer JP1.5, S1.1, S1.2
- net HIB: now also HIB.TP; no longer TP4.TP
- net LITE: now also LITE.1; no longer JP6.1
- net N$4: now also S1.A2; no longer S1.3, S1.4
- net N$5: now also SPKDAC.1; no longer JP7.1
- net N$7: now also SPKDAC.2; no longer JP7.2
- net PA0: now also U0RX.TP, UART0.1; no longer JP4.1
- net PA1: now also U0TX.TP, UART0.2; no longer JP4.2
- net PA2: now also SCK0.TP
- net PA3: now also CS0.TP
- net PA4: now also MOSI0.TP
- net PA5: now also MISO0.TP
- net PA6: now also DC0.TP
- net PA7: now also RST0.TP
- net PB4: now also FSS1.TP
- net PB5: now also SCLK1.TP
- net PC6: now also CCS.TP, U$1.19; no longer U$1.20
- net PC7: now also SDD.TP, U$1.20; no longer U$1.19
- net PD0: now also RI.TP, U$2.5; no longer U$2.8
- net PD1: now also KEY.TP, U$2.6; no longer U$2.7
- net PD2: now also PS.TP, U$2.7; no longer U$2.6
- net PD3: now also RSTG.TP, U$2.8; no longer U$2.5
- net PD4: now also U2RX.TP
- net PD5: now also U2TX.TP
- net PD7: now also NS.TP
- net PE0: now also U$1.11, Y+.TP; no longer U$1.14
- net PE1: now also U$1.12, X+.TP; no longer U$1.13
- net PE2: now also U$1.13, Y-.TP; no longer U$1.12
- net PE3: now also U$1.14, X-.TP; no longer U$1.11
- net PE4: now also MOSI1.TP
- net PE5: now also CS1.TP
- net PK0: now also U$1.18; no longer U$1.16, U1.18
- net PK1: no longer U1.19
- net PK2: now also U$1.16; no longer U$1.18, U1.20
- net PK4: now also SCL2.TP
- net PK5: now also SDA2.TP
- net PP0: now also U6RX.TP
- net PP1: now also U6TX.TP
- net SPKR+: now also SPKR.2; no longer JP3.2
- net SPKR-: now also SPKR.1; no longer JP3.1
- net TCK/SWCLK: now also JTAG.1; no longer JP1.1
- net TDI: now also JTAG.3; no longer JP1.3
- net TDO/SWO: now also JTAG.4; no longer JP1.4
- net TMS/SWDIO: now also JTAG.2; no longer JP1.2
- net VDDC: now also VDDC.TP; no longer TP5.TP
- net VREFA+: now also VREFA.TP; no longer TP1.TP
- net WAKE: now also WAKE.TP; no longer TP3.TP
Routing:
- net +3V3: track 0.00 -> 167.4 mm
- net +5V: track 0.00 -> 128.1 mm
- net PD7: track 0.00 -> 70.2 mm, vias 0 -> 1
- net PD5: track 0.00 -> 68.4 mm, vias 0 -> 1
- net PD4: track 0.00 -> 66.4 mm, vias 0 -> 1
- net PC7: track 0.00 -> 66.3 mm, vias 0 -> 1
- net PC6: track 0.00 -> 63.7 mm, vias 0 -> 1
- net PE0: track 0.00 -> 62.9 mm
- net PE1: track 0.00 -> 61.1 mm
- net PE2: track 0.00 -> 58.9 mm
- net PE3: track 0.00 -> 57.3 mm
- net PD3: track 0.00 -> 53.5 mm
- net PD2: track 0.00 -> 52.8 mm
- net PB4: track 0.00 -> 51.8 mm, vias 0 -> 1
- net PD1: track 0.00 -> 51.2 mm
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Other:
- board size 97.7 x 67.2 mm -> 116.6 x 67.2 mm

Commit message: Finished Final Board on EAGLE
Parts:
- added GND, GND2, GND3: TP_KEYSTONE500X, EE445L:P1.1MM
- C12, C13: value 4.7uF, Tantalum -> 4.7uF, T
- C16: value 1-4.7uF Tantalum -> 1-4.7uF, T
- S1: value MOMENTARY-SWITCH-SPST-SMD-6.2MM-TALL -> PTS636-G2.5; device SparkFun-Switches:TACTILE_SWITCH_SMD_6.2MM_TALL -> EE445L:PTS636-G
- moved U6RX 91.8 mm to (9.50, 3.90)
- moved U6TX 84.9 mm to (13.8, 3.90)
- moved C1 30.7 mm to (75.1, 33.6), turned to 90 degrees
- moved LITE 30.4 mm to (100.5, 34.9)
- moved C2 30.3 mm to (73.0, 33.6), turned to 90 degrees
- moved C3 29.8 mm to (70.9, 33.6), turned to 90 degrees
- moved C4 29.5 mm to (68.8, 33.6), turned to 90 degrees
- moved VDDC 6.07 mm to (36.3, 23.2)
- moved C8 4.13 mm to (40.9, 23.3), turned to 270 degrees
- moved C7 3.23 mm to (43.0, 23.3), turned to 270 degrees
- moved C6 2.73 mm to (45.1, 23.3), turned to 270 degrees
- moved R1 2.55 mm to (59.4, 45.8)
- moved C14 2.21 mm to (48.0, 6.13)
- moved R10 2.21 mm to (48.0, 10.3)
- moved C16 2.20 mm to (52.6, 13.0)
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Connections:
- removed net N$4: R6.2, S1.A2
- new net N$2: R6.2, S1.1
- net GND: now also GND.TP, GND2.TP, GND3.TP, S1.2; no longer S1.B2
Routing:
- net GND: track 2.00 -> 86.0 mm, vias 1 -> 16
- net +5V: track 128.1 -> 207.4 mm, vias 0 -> 3
- net PP0: track 0.00 -> 67.7 mm, vias 0 -> 1
- net PP1: track 0.00 -> 61.7 mm, vias 0 -> 1
- net PA2: track 4.24 -> 58.2 mm, vias 0 -> 1
- net PA0: track 0.00 -> 50.5 mm, vias 0 -> 1
- net PA5: track 4.24 -> 54.4 mm
- net PA4: track 4.23 -> 52.9 mm
- net PA7: track 4.24 -> 52.2 mm, vias 0 -> 2
- net PA1: track 0.00 -> 47.7 mm, vias 0 -> 1
- net PA3: track 4.24 -> 51.8 mm
- net PA6: track 4.24 -> 51.3 mm, vias 0 -> 2
- net PB5: track 27.2 -> 66.6 mm
- net LITE: track 0.00 -> 10.4 mm
- net +3V3: track 167.4 -> 173.2 mm
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- added copper zone on layer 1, net +3V3
- added copper zone on layer 16, net GND
