File: Phone_EE445L/Phone_EE445L.sch (EAGLE design)
At the start: 58 parts, among them IC1 LM4041CILPRCLP, Q1 NX5032GA, U2 TLV5616, U3 TPA751

Commit message: Continued finishing final board
Parts:
- removed JP2: (no value), EE445L:PINHD-1X2
- added CCS, CS0, CS1, DC0, FSS1, KEY, MISO0, MOSI0, MOSI1, NS, PS, RI, RST0, RSTG, SCK0, SCL2, SCLK1, SDA2, SDD, U0RX, U0TX, U2RX, U2TX, U6RX, U6TX, X+, X-, Y+, Y-: TP_KEYSTONE500X, EE445L:TP_KEYSTONE500X
- added PWR: (no value), EE445L:PINHD-1X2
- added SW1: (no value), EE445L:PUSHBUTTON
- S1: value (none) -> MOMENTARY-SWITCH-SPST-SMD-6.2MM-TALL; device EE445L:B3F-1052 -> SparkFun-Switches:MOMENTARY-SWITCH-SPST-SMD-6.2MM-TALL
- renumbered JP1 to JTAG, JP3 to SPKR, JP4 to UART0, JP5 to LCD-PWR, JP6 to LITE, JP7 to SPKDAC, TP1 to VREFA, TP2 to 3.3V, TP3 to WAKE, TP4 to HIB, TP5 to VDDC
Connections:
- net N$14 renamed HPF
- net N$15 renamed AMPIN
- net N$3 renamed WAKEVDD
- net N$6 renamed LCDPWR
- net N$9 renamed DACOUT
- removed net GNDA: C1.2, C2.2, C3.2, C4.2, U1G$16.GND@1, U1G$16.GND@2, U1G$16.GND@3, U1G$16.GND@4, U1G$16.GND@5, U1G$16.GND@6, U1G$18.GNDA
- removed net N$2: C1.1, C2.1, C3.1, C4.1, JP2.1, R2.2, R3.1, U1G$16.VDD@1, U1G$16.VDD@10, U1G$16.VDD@11, U1G$16.VDD@12, U1G$16.VDD@13, U1G$16.VDD@14, U1G$16.VDD@2, U1G$16.VDD@3, U1G$16.VDD@4, U1G$16.VDD@5, U1G$16.VDD@6, U1G$16.VDD@7, U1G$16.VDD@8, U1G$16.VDD@9, U1G$18.VDDA
- new net 5VIN: MICRO-USB.1, PWR.1, SW1.1
- net +3V3: now also C1.1, C2.1, C3.1, C4.1, R2.2, R3.1, U1G$16.VDD@1, U1G$16.VDD@10, U1G$16.VDD@11, U1G$16.VDD@12, U1G$16.VDD@13, U1G$16.VDD@14, U1G$16.VDD@2, U1G$16.VDD@3, U1G$16.VDD@4, U1G$16.VDD@5, U1G$16.VDD@6, U1G$16.VDD@7, U1G$16.VDD@8, U1G$16.VDD@9, U1G$18.VDDA; no longer JP2.2
- net +5V: now also PWR.2, SW1.6; no longer MICRO-USB.1
- net GND: now also C1.2, C2.2, C3.2, C4.2, S1.2, SW1.3, SW1.7, U1G$16.GND@1, U1G$16.GND@2, U1G$16.GND@3, U1G$16.GND@4, U1G$16.GND@5, U1G$16.GND@6, U1G$18.GNDA; no longer S1.S, S1.S1
- net N$4: now also S1.1; no longer S1.P, S1.P1
- net PA0: now also U0RX.TP
- net PA1: now also U0TX.TP
- net PA2: now also SCK0.TP
- net PA3: now also CS0.TP
- net PA4: now also MOSI0.TP
- net PA5: now also MISO0.TP
- net PA6: now also DC0.TP
- net PA7: now also RST0.TP
- net PB4: now also FSS1.TP
- net PB5: now also SCLK1.TP
- net PC6: now also CCS.TP, U$1.19; no longer U$1.20
- net PC7: now also SDD.TP, U$1.20; no longer U$1.19
- net PD0: now also RI.TP, U$2.5; no longer U$2.8
- net PD1: now also KEY.TP, U$2.6; no longer U$2.7
- net PD2: now also PS.TP, U$2.7; no longer U$2.6
- net PD3: now also RSTG.TP, U$2.8; no longer U$2.5
- net PD4: now also U2RX.TP
- net PD5: now also U2TX.TP
- net PD7: now also NS.TP
- net PE0: now also U$1.11, Y+.TP; no longer U$1.14
- net PE1: now also U$1.12, X+.TP; no longer U$1.13
- net PE2: now also U$1.13, Y-.TP; no longer U$1.12
- net PE3: now also U$1.14, X-.TP; no longer U$1.11
- net PE4: now also MOSI1.TP
- net PE5: now also CS1.TP
- net PK0: now also U$1.18; no longer U$1.16, U1G$10.PK0
- net PK1: no longer U1G$10.PK1
- net PK2: now also U$1.16; no longer U$1.18, U1G$10.PK2
- net PK4: now also SCL2.TP
- net PK5: now also SDA2.TP
- net PP0: now also U6RX.TP
- net PP1: now also U6TX.TP
Other:
- note added: "Fss1"
- moved on the sheet: C12, C13, D1, MICRO-USB, R9, U$4

Commit message: Finished Final Board on EAGLE
Parts:
- added GND, GND2, GND3: TP_KEYSTONE500X, EE445L:TP_KEYSTONE500X
- C12, C13: value 4.7uF, Tantalum -> 4.7uF, T
- C16: value 1-4.7uF Tantalum -> 1-4.7uF, T
- S1: value MOMENTARY-SWITCH-SPST-SMD-6.2MM-TALL -> PTS636-G2.5; device SparkFun-Switches:MOMENTARY-SWITCH-SPST-SMD-6.2MM-TALL -> EE445L:PTS636-G2.5
Connections:
- net GND: now also GND.TP, GND2.TP, GND3.TP
Other:
- moved on the sheet: C9
Changed lines of the file:
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@@
 <part name="SPKDAC" library="EE445L" deviceset="PINHD-1X2" device=""/>
 <part name="U$4" library="EE445L" deviceset="LM2937_HOR" device=""/>
-<part name="C12" library="EE445L" deviceset="CAPACITOR" device="050-024X044" value="4.7uF, Tantalum"/>
-<part name="C13" library="EE445L" deviceset="CAPACITOR" device="050-024X044" value="4.7uF, Tantalum"/>
+<part name="C12" library="EE445L" deviceset="CAPACITOR" device="050-024X044" value="4.7uF, T"/>
+<part name="C13" library="EE445L" deviceset="CAPACITOR" device="050-024X044" value="4.7uF, T"/>
 <part name="D1" library="SparkFun-LED" library_urn="urn:adsk.eagle:library:529" deviceset="LED" device="0603" package3d_urn="urn:adsk.eagle:package:39354/1"/>
 <part name="R9" library="rcl" library_urn="urn:adsk.eagle:library:334" deviceset="R-US_" device="R0805" package3d_urn="urn:adsk.eagle:package:23553/2"/>
@@
 <part name="C14" library="rcl" library_urn="urn:adsk.eagle:library:334" deviceset="C-US" device="C0805" package3d_urn="urn:adsk.eagle:package:23617/2" value="0.1uF"/>
 <part name="C15" library="rcl" library_urn="urn:adsk.eagle:library:334" deviceset="C-US" device="C0805" package3d_urn="urn:adsk.eagle:package:23617/2" value="0.1uF"/>
-<part name="C16" library="rcl" library_urn="urn:adsk.eagle:library:334" deviceset="C-US" device="C0805" package3d_urn="urn:adsk.eagle:package:23617/2" value="1-4.7uF Tantalum"/>
+<part name="C16" library="rcl" library_urn="urn:adsk.eagle:library:334" deviceset="C-US" device="C0805" package3d_urn="urn:adsk.eagle:package:23617/2" value="1-4.7uF, T"/>
 <part name="SUPPLY14" library="EE445L" deviceset="GND" device=""/>
 <part name="SUPPLY15" library="EE445L" deviceset="GND" device=""/>
@@
 <part name="MICRO-USB" library="EE445L" deviceset="ZX62D-B-5PA8(30)" device=""/>
 <part name="PWR" library="EE445L" deviceset="PINHD-1X2" device=""/>
-<part name="S1" library="SparkFun-Switches" library_urn="urn:adsk.eagle:library:535" deviceset="MOMENTARY-SWITCH-SPST" device="-SMD-6.2MM-TALL" package3d_urn="urn:adsk.eagle:package:40172/1"/>
+<part name="S1" library="EE445L" deviceset="PTS636-G2.5" device=""/>
 <part name="RI" library="EE445L" deviceset="TP" device="_KEYSTONE500X"/>
 <part name="KEY" library="EE445L" deviceset="TP" device="_KEYSTONE500X"/>
@@
 <part name="SDD" library="EE445L" deviceset="TP" device="_KEYSTONE500X"/>
 <part name="SW1" library="EE445L" deviceset="PUSHBUTTON" device=""/>
+<part name="GND2" library="EE445L" deviceset="TP" device="_KEYSTONE500X"/>
+<part name="GND" library="EE445L" deviceset="TP" device="_KEYSTONE500X"/>
+<part name="GND3" library="EE445L" deviceset="TP" device="_KEYSTONE500X"/>
+<part name="SUPPLY17" library="EE445L" deviceset="GND" device=""/>
 </parts>
 <sheets>
@@
 <attribute name="VALUE" x="89.662" y="-11.43" size="1.778" layer="96" rot="R90"/>
 </instance>
-<instance part="C9" gate="G$1" x="86.36" y="-20.32" smashed="yes">
-<attribute name="NAME" x="87.376" y="-19.685" size="1.778" layer="95"/>
-<attribute name="VALUE" x="87.376" y="-24.511" size="1.778" layer="96"/>
-</instance>
-<instance part="SUPPLY6" gate="GND" x="106.68" y="-35.56" smashed="yes">
-<attribute name="VALUE" x="102.235" y="-40.259" size="1.778" layer="96"/>
+<instance part="C9" gate="G$1" x="86.36" y="-22.86" smashed="yes">
+<attribute name="NAME" x="87.376" y="-22.225" size="1.778" layer="95"/>
+<attribute name="VALUE" x="87.376" y="-27.051" size="1.778" layer="96"/>
+</instance>
+<instance part="SUPPLY6" gate="GND" x="106.68" y="-40.64" smashed="yes">
+<attribute name="VALUE" x="102.235" y="-45.339" size="1.778" layer="96"/>
 </instance>
 <instance part="+3V1" gate="G$1" x="86.36" y="2.54" smashed="yes">
@@
 <attribute name="VALUE" x="38.735" y="35.941" size="1.778" layer="96"/>
 </instance>
-<instance part="S1" gate="G$1" x="106.68" y="-22.86" smashed="yes" rot="R270">
-<attribute name="NAME" x="108.204" y="-22.86" size="1.778" layer="95" font="vector" rot="R270" align="bottom-center"/>
-<attribute name="VALUE" x="112.268" y="-22.86" size="1.778" layer="96" font="vector" rot="R90" align="top-center"/>
+<instance part="S1" gate="A" x="106.68" y="-25.4" smashed="yes" rot="R270">
+<attribute name="NAME" x="108.204" y="-25.4" size="1.778" layer="95" font="vector" rot="R270" align="bottom-center"/>
+<attribute name="VALUE" x="112.268" y="-25.4" size="1.778" layer="96" font="vector" rot="R90" align="top-center"/>
 </instance>
 <instance part="CCS" gate="G$1" x="-53.34" y="50.8" smashed="yes" rot="R270">
@@
 <segment>
 <pinref part="SUPPLY6" gate="GND" pin="GND"/>
-<wire x1="106.68" y1="-27.94" x2="106.68" y2="-30.48" width="0.1524" layer="91"/>
-<wire x1="106.68" y1="-30.48" x2="106.68" y2="-33.02" width="0.1524" layer="91"/>
-<junction x="106.68" y="-30.48"/>
+<pinref part="S1" gate="A" pin="2"/>
+<wire x1="106.68" y1="-33.02" x2="106.68" y2="-35.56" width="0.1524" layer="91"/>
 <pinref part="C9" gate="G$1" pin="2"/>
-<wire x1="86.36" y1="-25.4" x2="86.36" y2="-30.48" width="0.1524" layer="91"/>
-<wire x1="86.36" y1="-30.48" x2="106.68" y2="-30.48" width="0.1524" layer="91"/>
-<pinref part="S1" gate="G$1" pin="2"/>
+<wire x1="106.68" y1="-35.56" x2="106.68" y2="-38.1" width="0.1524" layer="91"/>
+<wire x1="86.36" y1="-27.94" x2="86.36" y2="-35.56" width="0.1524" layer="91"/>
+<wire x1="86.36" y1="-35.56" x2="106.68" y2="-35.56" width="0.1524" layer="91"/>
+<junction x="106.68" y="-35.56"/>
 </segment>
 <segment>
@@
 <pinref part="R7" gate="G$1" pin="1"/>
 <pinref part="C9" gate="G$1" pin="1"/>
-<wire x1="86.36" y1="-17.78" x2="86.36" y2="-15.24" width="0.1524" layer="91"/>
+<wire x1="86.36" y1="-20.32" x2="86.36" y2="-15.24" width="0.1524" layer="91"/>
 <pinref part="R6" gate="G$1" pin="1"/>
 <wire x1="86.36" y1="-15.24" x2="86.36" y2="-12.7" width="0.1524" layer="91"/>
@@
 </segment>
 </net>
-<net name="N$4" class="0">
-<segment>
-<wire x1="106.68" y1="-17.78" x2="106.68" y2="-15.24" width="0.1524" layer="91"/>
-<pinref part="R6" gate="G$1" pin="2"/>
-<wire x1="101.6" y1="-15.24" x2="106.68" y2="-15.24" width="0.1524" layer="91"/>
-<pinref part="S1" gate="G$1" pin="1"/>
-</segment>
-</net>
 <net name="N$1" class="0">
 <segment>
@@
 <label x="-63.246" y="45.974" size="1.778" layer="95"/>
 <pinref part="SDD" gate="G$1" pin="TP"/>
+</segment>
+</net>
+<net name="N$2" class="0">
+<segment>
+<pinref part="R6" gate="G$1" pin="2"/>
+<wire x1="101.6" y1="-15.24" x2="106.68" y2="-15.24" width="0.1524" layer="91"/>
+<pinref part="S1" gate="A" pin="1"/>
+<wire x1="106.68" y1="-15.24" x2="106.68" y2="-17.78" width="0.1524" layer="91"/>
 </segment>
 </net>
@@
 <attribute name="TP_SIGNAL_NAME" x="-64.77" y="-67.31" size="1.778" layer="97" rot="R270"/>
 </instance>
+<instance part="GND2" gate="G$1" x="76.2" y="33.02" smashed="yes">
+<attribute name="NAME" x="74.93" y="34.29" size="1.778" layer="95"/>
+<attribute name="TP_SIGNAL_NAME" x="77.47" y="31.75" size="1.778" layer="97"/>
+</instance>
+<instance part="GND" gate="G$1" x="86.36" y="33.02" smashed="yes">
+<attribute name="NAME" x="85.09" y="34.29" size="1.778" layer="95"/>
+<attribute name="TP_SIGNAL_NAME" x="87.63" y="31.75" size="1.778" layer="97"/>
+</instance>
+<instance part="GND3" gate="G$1" x="96.52" y="33.02" smashed="yes">
+<attribute name="NAME" x="95.25" y="34.29" size="1.778" layer="95"/>
+<attribute name="TP_SIGNAL_NAME" x="97.79" y="31.75" size="1.778" layer="97"/>
+</instance>
+<instance part="SUPPLY17" gate="GND" x="86.36" y="17.78" smashed="yes">
+<attribute name="VALUE" x="81.915" y="13.081" size="1.778" layer="96"/>
+</instance>
 </instances>
 <busses>
@@
 <junction x="-15.24" y="27.94"/>
 </segment>
-</net>
+<segment>
+<pinref part="SUPPLY17" gate="GND" pin="GND"/>
+<pinref part="GND" gate="G$1" pin="TP"/>
+<wire x1="86.36" y1="20.32" x2="86.36" y2="25.4" width="0.1524" layer="91"/>
+<pinref part="GND3" gate="G$1" pin="TP"/>
+<wire x1="86.36" y1="25.4" x2="86.36" y2="30.48" width="0.1524" layer="91"/>
+<wire x1="96.52" y1="30.48" x2="96.52" y2="25.4" width="0.1524" layer="91"/>
+<wire x1="96.52" y1="25.4" x2="86.36" y2="25.4" width="0.1524" layer="91"/>
+<junction x="86.36" y="25.4"/>
+<pinref part="GND2" gate="G$1" pin="TP"/>
+<wire x1="76.2" y1="30.48" x2="76.2" y2="25.4" width="0.1524" layer="91"/>
+<wire x1="76.2" y1="25.4" x2="86.36" y2="25.4" width="0.1524" layer="91"/>
+</segment>
+</net>
